File: stm23-devkit.kicad_sch (KiCad schematic)
At the start: 26 parts, among them J1 Conn_01x04_Pin, J2 Conn_01x14, J3 USB_B_Micro, J5 Conn_01x14, SW1 SW_SPDT, U1 STM32F103C8T6, U2 AMS1117-3.3, Y2 16MHz

Commit message: Changes in schematic
Parts:
- removed J2, J5: Conn_01x14, symbol Connector_Generic:Conn_01x14
- added J2, J4: Conn_01x17, symbol Connector_Generic:Conn_01x17
- renumbered C6 to C1, C3 to C10, C8 to C11, C7 to C2, C11 to C3, C12 to C4, C13 to C5, C14 to C6, C15 to C7, C1 to C8, C2 to C9
Connections:
- net +3.3V: now also J2.1 (Pin_1), J4.1 (Pin_1)
- net GND: now also J4.2 (Pin_2)
- net PA10: now also J2.2 (Pin_2)
- net PA15: now also J4.3 (Pin_3)
- net PA3: now also J2.14 (Pin_14)
- net PA4: now also J2.13 (Pin_13)
- net PA5: now also J2.12 (Pin_12)
- net PA6: now also J2.11 (Pin_11)
- net PA7: now also J2.10 (Pin_10)
- net PA8: now also J2.4 (Pin_4)
- net PA9: now also J2.3 (Pin_3)
- net PB0: now also J2.7 (Pin_7)
- net PB1: now also J2.8 (Pin_8)
- net PB10: now also J2.6 (Pin_6)
- net PB11: now also J2.5 (Pin_5)
- net PB2: now also J2.9 (Pin_9)
- net PB3: now also J4.4 (Pin_4)
- net PB4: now also J4.5 (Pin_5)
- net PB5: now also J4.6 (Pin_6)
- net PB6: now also J4.7 (Pin_7)
- net PB7: now also J4.8 (Pin_8)
- net PB8: now also J4.9 (Pin_9)
- net PB9: now also J4.10 (Pin_10)
- net PC13: now also J4.11 (Pin_11)
- net PC14: now also J4.12 (Pin_12)
- net PC15: now also J4.13 (Pin_13)
- net PA0: now reaches U1.10 (PA0)
- net PA0: now also J2.17 (Pin_17)
- net PA1: now reaches U1.11 (PA1)
- net PA1: now also J2.16 (Pin_16)
- net PA2: now reaches U1.12 (PA2)
- net PA2: now also J2.15 (Pin_15)
- net PB12: now reaches U1.25 (PB12)
- net PB12: now also J4.14 (Pin_14)
- net PB13: now reaches U1.26 (PB13)
- net PB13: now also J4.15 (Pin_15)
- net PB14: now reaches U1.27 (PB14)
- net PB14: now also J4.16 (Pin_16)
- net PB15: now reaches U1.28 (PB15)
- net PB15: now also J4.17 (Pin_17)
- no-connect marks 6 -> 2
Other:
- note added: "Power Supply"
- moved on the sheet: C4, C5, Y2

Commit message: PCB created and organized
Parts:
- removed J3: USB_B_Micro, symbol Connector:USB_B_Micro
- removed R3: 1k5, symbol Device:R_Small
- added J5: MICROXNJ, MICROXNJ, symbol MICROXNJ:MICROXNJ
- added R4: 1k5, Resistor_SMD:R_0603_1608Metric, symbol Device:R_Small
- C1, C2: footprint (none) -> Capacitor_SMD:C_0805_2012Metric
- C10, C11, C3, C4, C5, C6, C7, C8, C9: footprint (none) -> Capacitor_SMD:C_0603_1608Metric
- C12: renamed from C4; footprint (none) -> Capacitor_SMD:C_0603_1608Metric
- C13: renamed from C5; footprint (none) -> Capacitor_SMD:C_0603_1608Metric
- D1: footprint (none) -> LED_SMD:LED_0603_1608Metric
- FB1: renamed from FB2; footprint (none) -> Inductor_SMD:L_0603_1608Metric
- J1: footprint (none) -> Connector_PinHeader_2.54mm:PinHeader_1x04_P2.54mm_Vertical
- J2, J4: footprint (none) -> Connector_PinHeader_2.54mm:PinHeader_1x17_P2.54mm_Vertical
- R1, R2: footprint (none) -> Resistor_SMD:R_0603_1608Metric
- SW1: footprint (none) -> Button_Switch_SMD:SW_SPDT_PCM12
- Y1: renamed from Y2; footprint (none) -> Crystal:Crystal_SMD_3225-4Pin_3.2x2.5mm
Connections:
- net +3.3V: now also R4.1
- net GND: now also J5.5
- net USB_D+: now also J5.3, R4.2
- net USB_D-: now also J5.2
- net VBUS: now also J5.1
- no-connect marks 2 -> 5
